Commit message: Update biqu_go1.urdf

File: Arm_URDF/biqu_go1.urdf (robot description, URDF)
Before this commit: robot robot, 22 links, 21 joints
Joints:
- joint j1: limit effort=1 velocity=20 -> lower=-0.863 upper=0.863 effort=9.72 velocity=1; type fixed -> revolute
- joint j2: limit effort=1 velocity=20 -> lower=-0.863 upper=0.863 effort=9.72 velocity=1; type fixed -> revolute
- joint j3: limit effort=1 velocity=20 -> lower=-0.863 upper=0.863 effort=9.72 velocity=1; type fixed -> revolute
